File: SM01.kicad_pcb (KiCad board)
At the start: 2 copper layers, 200 x 100 mm, 151 parts, among them J1 TRIG IN, J10 EXP3, J2 TRIG IN, J3 TRIG IN, J4 DC JACK, J5 TRIG IN, J6 VCA IN, J7 MIXOUT, J8 EXP1, J9 EXP2, Q1 2N3904, SW1 HOLD, SW10 DECAYSW2, SW11 DECAYSW3, SW13 DECAYSW4, SW14 OSCSW1, SW15 OSCSW2, SW16 OSCSW3, SW17 MUTE4, SW18 MUTE1, SW19 MUTE2, SW2 HOLD, SW20 MUTE3, SW21 MASTERSW, SW3 HOLD, SW4 ON, SW8 HOLD, SW9 DECAYSW1, U1 072, U10 072, U11 072, U2 072, U3 072, U4 7414, U5 7414, U6 7414, U8 072, U9 072

Commit message: may have made changes
Connections:
- U4 pad 14: Net-(C10-Pad1) -> Net-(U1-Pad6)
- U5 pad 14: Net-(C11-Pad1) -> Net-(U2-Pad6)
- U6 pad 14: Net-(C12-Pad1) -> Net-(U3-Pad6)
Routing:
- net Net-(U1-Pad6): track 2.54 -> 10.0 mm
- net Net-(C10-Pad1): track 33.4 -> 25.9 mm
- net Net-(U2-Pad6): track 2.54 -> 9.93 mm
- net Net-(C11-Pad1): track 33.2 -> 25.8 mm
- net Net-(U3-Pad6): track 2.54 -> 9.83 mm
- net Net-(C12-Pad1): track 32.9 -> 25.6 mm
Changed lines of the file:
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@@
-(kicad_pcb (version 20170123) (host pcbnew "(2017-09-01 revision 8d1475135)-makepkg")
+(kicad_pcb (version 20170123) (host pcbnew "(2017-06-11 revision d5e8572)-master")
   (general
+    (links 300)
+    (no_connects 3)
+    (area -2.5 -100.075001 200.075001 2.5)
     (thickness 1.6)
     (drawings 8)
@@
       (usegerberattributes true)
       (usegerberadvancedattributes true)
-      (creategerberjobfile true)
       (excludeedgelayer true)
       (linewidth 0.100000)
@@
     )
     (pad 14 thru_hole oval (at 7.62 0 90) (size 1.6 1.6) (drill 0.8) (layers *.Cu *.Mask)
-      (net 85 "Net-(C10-Pad1)"))
+      (net 114 "Net-(U1-Pad6)"))
     (pad 7 thru_hole oval (at 0 -15.24 90) (size 1.6 1.6) (drill 0.8) (layers *.Cu *.Mask)
       (net 2 GND))
@@
       (net 2 GND))
     (pad 14 thru_hole oval (at 7.62 0 90) (size 1.6 1.6) (drill 0.8) (layers *.Cu *.Mask)
-      (net 81 "Net-(C12-Pad1)"))
+      (net 116 "Net-(U3-Pad6)"))
     (model ${KISYS3DMOD}/Housings_DIP.3dshapes/DIP-14_W7.62mm.wrl
       (at (xyz 0 0 0))
@@
     )
     (pad 14 thru_hole oval (at 7.62 0 90) (size 1.6 1.6) (drill 0.8) (layers *.Cu *.Mask)
-      (net 84 "Net-(C11-Pad1)"))
+      (net 115 "Net-(U2-Pad6)"))
     (pad 7 thru_hole oval (at 0 -15.24 90) (size 1.6 1.6) (drill 0.8) (layers *.Cu *.Mask)
       (net 2 GND))
@@
   (segment (start 113.284 -27.432) (end 113.284 -46.99) (width 0.25) (layer F.Cu) (net 81))
   (via (at 113.284 -46.99) (size 0.8) (drill 0.4) (layers F.Cu B.Cu) (net 81))
-  (segment (start 113.284 -24.638) (end 106.018 -24.638) (width 0.25) (layer B.Cu) (net 81))
-  (segment (start 106.018 -24.638) (end 106 -24.62) (width 0.25) (layer B.Cu) (net 81))
   (segment (start 113.284 -27.432) (end 113.284 -24.638) (width 0.25) (layer F.Cu) (net 81))
   (via (at 113.284 -24.638) (size 0.8) (drill 0.4) (layers F.Cu B.Cu) (net 81))
@@
   (segment (start 73.406 -24.638) (end 73.406 -25.203685) (width 0.25) (layer F.Cu) (net 84))
   (segment (start 73.406 -25.203685) (end 73.406 -27.94) (width 0.25) (layer F.Cu) (net 84))
-  (segment (start 66 -24.62) (end 73.388 -24.62) (width 0.25) (layer B.Cu) (net 84))
-  (segment (start 73.388 -24.62) (end 73.406 -24.638) (width 0.25) (layer B.Cu) (net 84))
   (via (at 73.406 -24.638) (size 0.8) (drill 0.4) (layers F.Cu B.Cu) (net 84))
+  (segment (start 73.388 -24.62) (end 73.406 -24.638) (width 0.25) (layer B.Cu) (net 84))
   (segment (start 33.528 -24.638) (end 33.528 -28.956) (width 0.25) (layer F.Cu) (net 85))
   (via (at 33.528 -24.638) (size 0.8) (drill 0.4) (layers F.Cu B.Cu) (net 85))
-  (segment (start 26 -24.62) (end 33.51 -24.62) (width 0.25) (layer B.Cu) (net 85))
   (segment (start 33.51 -24.62) (end 33.528 -24.638) (width 0.25) (layer B.Cu) (net 85))
   (segment (start 33.528 -28.956) (end 33.528 -46.99) (width 0.25) (layer F.Cu) (net 85))
@@
   (segment (start 102.46 -69) (end 102.46 -66.85) (width 0.25) (layer F.Cu) (net 95))
   (segment (start 102.46 -66.85) (end 102.5 -66.81) (width 0.25) (layer F.Cu) (net 95))
-  (segment (start 135.89 -24.13) (end 136.017 -24.257) (width 0.25) (layer B.Cu) (net 109))
-  (segment (start 131.826 -24.13) (end 135.89 -24.13) (width 0.25) (layer B.Cu) (net 109))
-  (segment (start 136.0805 -24.3205) (end 136.017 -24.257) (width 0.25) (layer F.Cu) (net 109))
-  (segment (start 136.0805 -32.893) (end 136.0805 -24.3205) (width 0.25) (layer F.Cu) (net 109))
-  (via (at 136.017 -24.257) (size 0.8) (drill 0.4) (layers F.Cu B.Cu) (net 109))
-  (segment (start 153.416 -33.02) (end 136.2075 -33.02) (width 0.25) (layer B.Cu) (net 109))
-  (segment (start 136.2075 -33.02) (end 136.0805 -32.893) (width 0.25) (layer B.Cu) (net 109))
-  (via (at 136.0805 -32.893) (size 0.8) (drill 0.4) (layers F.Cu B.Cu) (net 109))
-  (segment (start 153.2255 -42.9895) (end 153.2255 -33.2105) (width 0.25) (layer F.Cu) (net 109))
-  (via (at 153.416 -33.02) (size 0.8) (drill 0.4) (layers F.Cu B.Cu) (net 109))
-  (segment (start 153.2255 -33.2105) (end 153.416 -33.02) (width 0.25) (layer F.Cu) (net 109))
-  (segment (start 155.194 -42.926) (end 153.289 -42.926) (width 0.25) (layer B.Cu) (net 109))
-  (segment (start 153.289 -42.926) (end 153.2255 -42.9895) (width 0.25) (layer B.Cu) (net 109))
-  (via (at 153.2255 -42.9895) (size 0.8) (drill 0.4) (layers F.Cu B.Cu) (net 109))
-  (segment (start 128.524 -21.59) (end 127 -21.59) (width 0.5) (layer B.Cu) (net 109))
-  (segment (start 129.54 -20.574) (end 128.524 -21.59) (width 0.5) (layer B.Cu) (net 109))
-  (segment (start 131.318 -20.574) (end 129.54 -20.574) (width 0.5) (layer B.Cu) (net 109))
-  (segment (start 131.826 -24.13) (end 131.826 -21.082) (width 0.5) (layer F.Cu) (net 109))
-  (segment (start 131.826 -21.082) (end 131.318 -20.574) (width 0.5) (layer F.Cu) (net 109))
   (segment (start 25 -69) (end 30.392 -69) (width 0.25) (layer B.Cu) (net 96))
   (segment (start 30.392 -69) (end 30.734 -69.342) (width 0.25) (layer B.Cu) (net 96))
@@
   (via (at 20.574 -41.91) (size 0.8) (drill 0.4) (layers F.Cu B.Cu) (net 108))
   (segment (start 9.999837 -42.012243) (end 12.539837 -42.012243) (width 0.25) (layer B.Cu) (net 108))
+  (segment (start 135.89 -24.13) (end 136.017 -24.257) (width 0.25) (layer B.Cu) (net 109))
+  (segment (start 131.826 -24.13) (end 135.89 -24.13) (width 0.25) (layer B.Cu) (net 109))
+  (segment (start 136.0805 -24.3205) (end 136.017 -24.257) (width 0.25) (layer F.Cu) (net 109))
+  (segment (start 136.0805 -32.893) (end 136.0805 -24.3205) (width 0.25) (layer F.Cu) (net 109))
+  (via (at 136.017 -24.257) (size 0.8) (drill 0.4) (layers F.Cu B.Cu) (net 109))
+  (segment (start 153.416 -33.02) (end 136.2075 -33.02) (width 0.25) (layer B.Cu) (net 109))
+  (segment (start 136.2075 -33.02) (end 136.0805 -32.893) (width 0.25) (layer B.Cu) (net 109))
+  (via (at 136.0805 -32.893) (size 0.8) (drill 0.4) (layers F.Cu B.Cu) (net 109))
+  (segment (start 153.2255 -42.9895) (end 153.2255 -33.2105) (width 0.25) (layer F.Cu) (net 109))
+  (via (at 153.416 -33.02) (size 0.8) (drill 0.4) (layers F.Cu B.Cu) (net 109))
+  (segment (start 153.2255 -33.2105) (end 153.416 -33.02) (width 0.25) (layer F.Cu) (net 109))
+  (segment (start 155.194 -42.926) (end 153.289 -42.926) (width 0.25) (layer B.Cu) (net 109))
+  (segment (start 153.289 -42.926) (end 153.2255 -42.9895) (width 0.25) (layer B.Cu) (net 109))
+  (via (at 153.2255 -42.9895) (size 0.8) (drill 0.4) (layers F.Cu B.Cu) (net 109))
+  (segment (start 128.524 -21.59) (end 127 -21.59) (width 0.5) (layer B.Cu) (net 109))
+  (segment (start 129.54 -20.574) (end 128.524 -21.59) (width 0.5) (layer B.Cu) (net 109))
+  (segment (start 131.318 -20.574) (end 129.54 -20.574) (width 0.5) (layer B.Cu) (net 109))
+  (segment (start 131.826 -24.13) (end 131.826 -21.082) (width 0.5) (layer F.Cu) (net 109))
+  (segment (start 131.826 -21.082) (end 131.318 -20.574) (width 0.5) (layer F.Cu) (net 109))
   (segment (start 167.459837 -86.012243) (end 167.459837 -68.762243) (width 0.25) (layer F.Cu) (net 109))
   (segment (start 155.194 -42.926) (end 156.21 -41.91) (width 0.25) (layer B.Cu) (net 109))
@@
   (segment (start 32.258 -79.756) (end 33.782 -78.232) (width 0.25) (layer F.Cu) (net 113))
   (segment (start 33.782 -78.232) (end 33.782 -77.216) (width 0.25) (layer F.Cu) (net 113))
+  (segment (start 26 -24.62) (end 33.51 -24.62) (width 0.25) (layer B.Cu) (net 114))
   (segment (start 19.92 -76.62) (end 21.05137 -76.62) (width 0.25) (layer B.Cu) (net 114))
   (segment (start 21.05137 -76.62) (end 22.46 -76.62) (width 0.25) (layer B.Cu) (net 114))
+  (segment (start 66 -24.62) (end 73.388 -24.62) (width 0.25) (layer B.Cu) (net 115))
   (segment (start 59.92 -76.62) (end 62.46 -76.62) (width 0.25) (layer B.Cu) (net 115))
+  (segment (start 113.284 -24.638) (end 106.018 -24.638) (width 0.25) (layer B.Cu) (net 116))
+  (segment (start 106.018 -24.638) (end 106 -24.62) (width 0.25) (layer B.Cu) (net 116))
   (segment (start 99.92 -76.62) (end 101.05137 -76.62) (width 0.25) (layer B.Cu) (net 116))
   (segment (start 101.05137 -76.62) (end 102.46 -76.62) (width 0.25) (layer B.Cu) (net 116))
