File: SM01.sch (KiCad schematic (older format))
At the start: 151 parts, among them J1 TRIG IN, J10 EXP3, J2 TRIG IN, J3 TRIG IN, J4 DC JACK, J5 TRIG IN, J6 VCA IN, J7 MIXOUT, J8 EXP1, J9 EXP2, Q1 2N3904, SW1 HOLD, SW10 DECAYSW2, SW11 DECAYSW3, SW13 DECAYSW4, SW14 OSCSW1, SW15 OSCSW2, SW16 OSCSW3, SW17 MUTE4, SW18 MUTE1, SW19 MUTE2, SW2 HOLD, SW20 MUTE3, SW21 MASTERSW, SW3 HOLD, SW4 ON, SW8 HOLD, SW9 DECAYSW1, U1 072, U10 072, U11 072, U2 072, U3 072, U4 7414, U5 7414, U6 7414, U8 072, U9 072

Commit message: added gbr - sent file in -HOPE IT WORKS!
Changed lines of the file:
@@
 L GND #PWR07
 U 1 1 599C70BA
-P 1100 1550
-F 0 "#PWR07" H 1100 1300 50  0001 C CNN
-F 1 "GND" H 900 1450 50  0000 C CNN
-F 2 "" H 1100 1550 50  0001 C CNN
-F 3 "" H 1100 1550 50  0001 C CNN
-	1    1100 1550
+P 1150 1550
+F 0 "#PWR07" H 1150 1300 50  0001 C CNN
+F 1 "GND" H 950 1450 50  0000 C CNN
+F 2 "" H 1150 1550 50  0001 C CNN
+F 3 "" H 1150 1550 50  0001 C CNN
+	1    1150 1550
 	1    0    0    -1
 $EndComp
@@
 L GND #PWR09
 U 1 1 59A1E024
-P 8450 9950
-F 0 "#PWR09" H 8450 9700 50  0001 C CNN
-F 1 "GND" H 8455 9777 50  0000 C CNN
-F 2 "" H 8450 9950 50  0001 C CNN
-F 3 "" H 8450 9950 50  0001 C CNN
-	1    8450 9950
+P 8450 9900
+F 0 "#PWR09" H 8450 9650 50  0001 C CNN
+F 1 "GND" H 8455 9727 50  0000 C CNN
+F 2 "" H 8450 9900 50  0001 C CNN
+F 3 "" H 8450 9900 50  0001 C CNN
+	1    8450 9900
 	1    0    0    -1
 $EndComp
@@
 L +5V #PWR012
 U 1 1 59A2ED70
-P 1500 2150
-F 0 "#PWR012" H 1500 2000 50  0001 C CNN
-F 1 "+5V" H 1515 2323 50  0000 C CNN
-F 2 "" H 1500 2150 50  0001 C CNN
-F 3 "" H 1500 2150 50  0001 C CNN
-	1    1500 2150
+P 1600 2150
+F 0 "#PWR012" H 1600 2000 50  0001 C CNN
+F 1 "+5V" H 1615 2323 50  0000 C CNN
+F 2 "" H 1600 2150 50  0001 C CNN
+F 3 "" H 1600 2150 50  0001 C CNN
+	1    1600 2150
 	1    0    0    -1
 $EndComp
@@
 L GND #PWR029
 U 1 1 59AD1FC9
-P 4400 9300
-F 0 "#PWR029" H 4400 9050 50  0001 C CNN
-F 1 "GND" H 4405 9127 50  0000 C CNN
-F 2 "" H 4400 9300 50  0001 C CNN
-F 3 "" H 4400 9300 50  0001 C CNN
-	1    4400 9300
+P 4400 9250
+F 0 "#PWR029" H 4400 9000 50  0001 C CNN
+F 1 "GND" H 4405 9077 50  0000 C CNN
+F 2 "" H 4400 9250 50  0001 C CNN
+F 3 "" H 4400 9250 50  0001 C CNN
+	1    4400 9250
 	1    0    0    -1
 $EndComp
@@
 	10200 9100 10150 9100
 Wire Wire Line
-	1600 2150 1500 2150
-Wire Wire Line
 	1750 2550 1750 2600
 Wire Wire Line
@@
 	12450 2450 12450 9450
 Wire Wire Line
-	4400 9250 4400 9300
-Wire Wire Line
 	5900 9100 5900 9450
 Wire Wire Line
@@
 	8650 9100 9300 9100
 Wire Wire Line
-	8450 9900 8450 9950
-Wire Wire Line
 	6650 4200 6650 4500
 Wire Wire Line
@@
 Connection ~ 10250 6400
 Wire Wire Line
-	1100 1550 1150 1550
-Wire Wire Line
 	1600 1550 1650 1550

Commit message: may have made changes
Other:
- note added: "WHY PIN 14?????? AHHHH!!!\n"
